File: hardware/vin_display_hdsp2000_x20/displays2.kicad_sch (KiCad schematic)
At the start: 22 parts, among them U15 HDSP-2000, U16 HDSP-2000, U17 HDSP-2000, U18 HDSP-2000, U19 HDSP-2000, U20 HDSP-2000, U21 HDSP-2000, U22 HDSP-2000, U23 HDSP-2000, U24 HDSP-2000

Commit message: route hdsp2000_x20 board
Parts:
- C33, C34, C35, C36, C37, C38, C39, C40, C41, C42: footprint (none) -> Capacitor_SMD:C_0603_1608Metric
- JP1: footprint (none) -> components:Solder_jumber_3pad
- R14: footprint (none) -> Resistor_SMD:R_0603_1608Metric
- U15, U16, U17, U18, U19, U20, U21, U22, U23, U24: footprint (none) -> components:HDSP_DIP12
Changed lines of the file:
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@@
       (effects (font (size 1.27 1.27)))
     )
-    (property "Footprint" "" (at 213.995 64.135 0)
+    (property "Footprint" "components:HDSP_DIP12" (at 213.995 64.135 0)
       (effects (font (size 1.27 1.27)) hide)
     )
@@
       (effects (font (size 1.27 1.27)))
     )
-    (property "Footprint" "" (at 255.905 151.003 90)
+    (property "Footprint" "Resistor_SMD:R_0603_1608Metric" (at 255.905 151.003 90)
       (effects (font (size 1.27 1.27)) hide)
     )
@@
       (effects (font (size 1.27 1.27)))
     )
-    (property "Footprint" "" (at 269.875 63.1698 0)
+    (property "Footprint" "Capacitor_SMD:C_0603_1608Metric" (at 269.875 63.1698 0)
       (effects (font (size 1.27 1.27)) hide)
     )
@@
       (effects (font (size 1.27 1.27)))
     )
-    (property "Footprint" "" (at 42.545 61.2648 0)
+    (property "Footprint" "Capacitor_SMD:C_0603_1608Metric" (at 42.545 61.2648 0)
       (effects (font (size 1.27 1.27)) hide)
     )
@@
       (effects (font (size 1.27 1.27)))
     )
-    (property "Footprint" "" (at 269.875 98.0948 0)
+    (property "Footprint" "Capacitor_SMD:C_0603_1608Metric" (at 269.875 98.0948 0)
       (effects (font (size 1.27 1.27)) hide)
     )
@@
       (effects (font (size 1.27 1.27)))
     )
-    (property "Footprint" "" (at 213.995 90.805 0)
+    (property "Footprint" "components:HDSP_DIP12" (at 213.995 90.805 0)
       (effects (font (size 1.27 1.27)) hide)
     )
@@
       (effects (font (size 1.27 1.27)) (justify left) hide)
     )
-    (property "Footprint" "" (at 110.49 29.21 0)
+    (property "Footprint" "components:Solder_jumber_3pad" (at 110.49 29.21 0)
       (effects (font (size 1.27 1.27)) hide)
     )
@@
       (effects (font (size 1.27 1.27)))
     )
-    (property "Footprint" "" (at 269.875 51.7398 0)
+    (property "Footprint" "Capacitor_SMD:C_0603_1608Metric" (at 269.875 51.7398 0)
       (effects (font (size 1.27 1.27)) hide)
     )
@@
       (effects (font (size 1.27 1.27)))
     )
-    (property "Footprint" "" (at 83.185 90.17 0)
+    (property "Footprint" "components:HDSP_DIP12" (at 83.185 90.17 0)
       (effects (font (size 1.27 1.27)) hide)
     )
@@
       (effects (font (size 1.27 1.27)))
     )
-    (property "Footprint" "" (at 83.185 63.5 0)
+    (property "Footprint" "components:HDSP_DIP12" (at 83.185 63.5 0)
       (effects (font (size 1.27 1.27)) hide)
     )
@@
       (effects (font (size 1.27 1.27)))
     )
-    (property "Footprint" "" (at 83.185 116.84 0)
+    (property "Footprint" "components:HDSP_DIP12" (at 83.185 116.84 0)
       (effects (font (size 1.27 1.27)) hide)
     )
@@
       (effects (font (size 1.27 1.27)))
     )
-    (property "Footprint" "" (at 269.875 74.5998 0)
+    (property "Footprint" "Capacitor_SMD:C_0603_1608Metric" (at 269.875 74.5998 0)
       (effects (font (size 1.27 1.27)) hide)
     )
@@
       (effects (font (size 1.27 1.27)))
     )
-    (property "Footprint" "" (at 42.545 96.1898 0)
+    (property "Footprint" "Capacitor_SMD:C_0603_1608Metric" (at 42.545 96.1898 0)
       (effects (font (size 1.27 1.27)) hide)
     )
@@
       (effects (font (size 1.27 1.27)))
     )
-    (property "Footprint" "" (at 213.995 117.475 0)
+    (property "Footprint" "components:HDSP_DIP12" (at 213.995 117.475 0)
       (effects (font (size 1.27 1.27)) hide)
     )
@@
       (effects (font (size 1.27 1.27)))
     )
-    (property "Footprint" "" (at 42.545 72.6948 0)
+    (property "Footprint" "Capacitor_SMD:C_0603_1608Metric" (at 42.545 72.6948 0)
       (effects (font (size 1.27 1.27)) hide)
     )
@@
       (effects (font (size 1.27 1.27)))
     )
-    (property "Footprint" "" (at 213.995 37.465 0)
+    (property "Footprint" "components:HDSP_DIP12" (at 213.995 37.465 0)
       (effects (font (size 1.27 1.27)) hide)
     )
@@
       (effects (font (size 1.27 1.27)))
     )
-    (property "Footprint" "" (at 42.545 49.8348 0)
+    (property "Footprint" "Capacitor_SMD:C_0603_1608Metric" (at 42.545 49.8348 0)
       (effects (font (size 1.27 1.27)) hide)
     )
@@
       (effects (font (size 1.27 1.27)))
     )
-    (property "Footprint" "" (at 213.995 144.145 0)
+    (property "Footprint" "components:HDSP_DIP12" (at 213.995 144.145 0)
       (effects (font (size 1.27 1.27)) hide)
     )
@@
       (effects (font (size 1.27 1.27)))
     )
-    (property "Footprint" "" (at 269.875 86.6648 0)
+    (property "Footprint" "Capacitor_SMD:C_0603_1608Metric" (at 269.875 86.6648 0)
       (effects (font (size 1.27 1.27)) hide)
     )
@@
       (effects (font (size 1.27 1.27)))
     )
-    (property "Footprint" "" (at 83.185 143.51 0)
+    (property "Footprint" "components:HDSP_DIP12" (at 83.185 143.51 0)
       (effects (font (size 1.27 1.27)) hide)
     )
@@
       (effects (font (size 1.27 1.27)))
     )
-    (property "Footprint" "" (at 42.545 84.7598 0)
+    (property "Footprint" "Capacitor_SMD:C_0603_1608Metric" (at 42.545 84.7598 0)
       (effects (font (size 1.27 1.27)) hide)
     )
@@
       (effects (font (size 1.27 1.27)))
     )
-    (property "Footprint" "" (at 83.185 36.83 0)
-      (effects (font (size 1.27 1.27)) hide)
-    )
+    (property "Footprint" "components:HDSP_DIP12" (at 83.185 36.83 0)
+      (effects (font (size 1.27 1.27)) hide)
+    )
