File: hardware/vin_display_hdsp2000_x20/displays.kicad_sch (KiCad schematic)
At the start: 31 parts, among them Q2 DMP2022LSS, Q3 DMP2022LSS, Q4 DMP2022LSS, Q5 DMP2022LSS, Q6 DMP2022LSS, U10 HDSP-2000, U11 HDSP-2000, U12 HDSP-2000, U13 HDSP-2000, U14 HDSP-2000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

Commit message: route hdsp2000_x20 board
Parts:
- C23, C24, C25, C26, C27, C28, C29, C30, C31, C32: footprint (none) -> Capacitor_SMD:C_0603_1608Metric
- Q2, Q3, Q4, Q5, Q6: footprint (none) -> components:SO8_MOSFET_S3G1D4
- R15, R16, R17, R18, R19, R20: footprint (none) -> Resistor_SMD:R_0603_1608Metric
- U10, U11, U12, U13, U14, U5, U6, U7, U8, U9: footprint (none) -> components:HDSP_DIP12
Changed lines of the file:
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@@
       (effects (font (size 1.27 1.27)))
     )
-    (property "Footprint" "" (at 78.105 35.56 0)
+    (property "Footprint" "components:HDSP_DIP12" (at 78.105 35.56 0)
       (effects (font (size 1.27 1.27)) hide)
     )
@@
       (effects (font (size 1.27 1.27)))
     )
-    (property "Footprint" "" (at 78.105 115.57 0)
+    (property "Footprint" "components:HDSP_DIP12" (at 78.105 115.57 0)
       (effects (font (size 1.27 1.27)) hide)
     )
@@
       (effects (font (size 1.27 1.27)))
     )
-    (property "Footprint" "" (at 78.105 88.9 0)
+    (property "Footprint" "components:HDSP_DIP12" (at 78.105 88.9 0)
       (effects (font (size 1.27 1.27)) hide)
     )
@@
       (effects (font (size 1.27 1.27)) (justify left))
     )
-    (property "Footprint" "" (at 138.43 153.67 0)
+    (property "Footprint" "components:SO8_MOSFET_S3G1D4" (at 138.43 153.67 0)
       (effects (font (size 1.27 1.27)) hide)
     )
@@
       (effects (font (size 1.27 1.27)))
     )
-    (property "Footprint" "" (at 215.9 33.655 0)
+    (property "Footprint" "components:HDSP_DIP12" (at 215.9 33.655 0)
       (effects (font (size 1.27 1.27)) hide)
     )
@@
       (effects (font (size 1.27 1.27)) (justify left))
     )
-    (property "Footprint" "" (at 148.082 144.78 90)
+    (property "Footprint" "Resistor_SMD:R_0603_1608Metric" (at 148.082 144.78 90)
       (effects (font (size 1.27 1.27)) hide)
     )
@@
       (effects (font (size 1.27 1.27)))
     )
-    (property "Footprint" "" (at 215.9 113.665 0)
+    (property "Footprint" "components:HDSP_DIP12" (at 215.9 113.665 0)
       (effects (font (size 1.27 1.27)) hide)
     )
@@
       (effects (font (size 1.27 1.27)))
     )
-    (property "Footprint" "" (at 40.005 84.1248 0)
+    (property "Footprint" "Capacitor_SMD:C_0603_1608Metric" (at 40.005 84.1248 0)
       (effects (font (size 1.27 1.27)) hide)
     )
@@
       (effects (font (size 1.27 1.27)) (justify left))
     )
-    (property "Footprint" "" (at 137.795 101.6 0)
+    (property "Footprint" "components:SO8_MOSFET_S3G1D4" (at 137.795 101.6 0)
       (effects (font (size 1.27 1.27)) hide)
     )
@@
       (effects (font (size 1.27 1.27)) (justify left))
     )
-    (property "Footprint" "" (at 136.525 48.895 0)
+    (property "Footprint" "components:SO8_MOSFET_S3G1D4" (at 136.525 48.895 0)
       (effects (font (size 1.27 1.27)) hide)
     )
@@
       (effects (font (size 1.27 1.27)))
     )
-    (property "Footprint" "" (at 267.335 67.6148 0)
+    (property "Footprint" "Capacitor_SMD:C_0603_1608Metric" (at 267.335 67.6148 0)
       (effects (font (size 1.27 1.27)) hide)
     )
@@
       (effects (font (size 1.27 1.27)))
     )
-    (property "Footprint" "" (at 40.005 72.0598 0)
+    (property "Footprint" "Capacitor_SMD:C_0603_1608Metric" (at 40.005 72.0598 0)
       (effects (font (size 1.27 1.27)) hide)
     )
@@
       (effects (font (size 1.27 1.27)) (justify left))
     )
-    (property "Footprint" "" (at 138.43 127.635 0)
+    (property "Footprint" "components:SO8_MOSFET_S3G1D4" (at 138.43 127.635 0)
       (effects (font (size 1.27 1.27)) hide)
     )
@@
       (effects (font (size 1.27 1.27)))
     )
-    (property "Footprint" "" (at 40.005 60.6298 0)
+    (property "Footprint" "Capacitor_SMD:C_0603_1608Metric" (at 40.005 60.6298 0)
       (effects (font (size 1.27 1.27)) hide)
     )
@@
       (effects (font (size 1.27 1.27)) (justify left))
     )
-    (property "Footprint" "" (at 146.177 40.005 90)
+    (property "Footprint" "Resistor_SMD:R_0603_1608Metric" (at 146.177 40.005 90)
       (effects (font (size 1.27 1.27)) hide)
     )
@@
       (effects (font (size 1.27 1.27)))
     )
-    (property "Footprint" "" (at 267.335 79.6798 0)
+    (property "Footprint" "Capacitor_SMD:C_0603_1608Metric" (at 267.335 79.6798 0)
       (effects (font (size 1.27 1.27)) hide)
     )
@@
       (effects (font (size 1.27 1.27)))
     )
-    (property "Footprint" "" (at 215.9 86.995 0)
+    (property "Footprint" "components:HDSP_DIP12" (at 215.9 86.995 0)
       (effects (font (size 1.27 1.27)) hide)
     )
@@
       (effects (font (size 1.27 1.27)) (justify left))
     )
-    (property "Footprint" "" (at 137.16 75.565 0)
+    (property "Footprint" "components:SO8_MOSFET_S3G1D4" (at 137.16 75.565 0)
       (effects (font (size 1.27 1.27)) hide)
     )
@@
       (effects (font (size 1.27 1.27)))
     )
-    (property "Footprint" "" (at 78.105 62.23 0)
+    (property "Footprint" "components:HDSP_DIP12" (at 78.105 62.23 0)
       (effects (font (size 1.27 1.27)) hide)
     )
@@
       (effects (font (size 1.27 1.27)))
     )
-    (property "Footprint" "" (at 267.335 44.7548 0)
+    (property "Footprint" "Capacitor_SMD:C_0603_1608Metric" (at 267.335 44.7548 0)
       (effects (font (size 1.27 1.27)) hide)
     )
@@
       (effects (font (size 1.27 1.27)))
     )
-    (property "Footprint" "" (at 40.005 95.5548 0)
+    (property "Footprint" "Capacitor_SMD:C_0603_1608Metric" (at 40.005 95.5548 0)
       (effects (font (size 1.27 1.27)) hide)
     )
@@
       (effects (font (size 1.27 1.27)))
     )
-    (property "Footprint" "" (at 215.9 140.335 0)
+    (property "Footprint" "components:HDSP_DIP12" (at 215.9 140.335 0)
       (effects (font (size 1.27 1.27)) hide)
     )
@@
       (effects (font (size 1.27 1.27)) (justify left))
     )
-    (property "Footprint" "" (at 147.447 92.71 90)
+    (property "Footprint" "Resistor_SMD:R_0603_1608Metric" (at 147.447 92.71 90)
       (effects (font (size 1.27 1.27)) hide)
     )
@@
       (effects (font (size 1.27 1.27)))
     )
-    (property "Footprint" "" (at 215.9 60.325 0)
+    (property "Footprint" "components:HDSP_DIP12" (at 215.9 60.325 0)
       (effects (font (size 1.27 1.27)) hide)
     )
@@
       (effects (font (size 1.27 1.27)))
     )
-    (property "Footprint" "" (at 267.335 91.1098 0)
+    (property "Footprint" "Capacitor_SMD:C_0603_1608Metric" (at 267.335 91.1098 0)
       (effects (font (size 1.27 1.27)) hide)
     )
@@
       (effects (font (size 1.27 1.27)) (justify left))
     )
-    (property "Footprint" "" (at 148.082 118.745 90)
+    (property "Footprint" "Resistor_SMD:R_0603_1608Metric" (at 148.082 118.745 90)
       (effects (font (size 1.27 1.27)) hide)
     )
@@
       (effects (font (size 1.27 1.27)))
     )
-    (property "Footprint" "" (at 267.335 56.1848 0)
+    (property "Footprint" "Capacitor_SMD:C_0603_1608Metric" (at 267.335 56.1848 0)
       (effects (font (size 1.27 1.27)) hide)
     )
@@
       (effects (font (size 1.27 1.27)) (justify left))
     )
-    (property "Footprint" "" (at 228.727 151.765 90)
+    (property "Footprint" "Resistor_SMD:R_0603_1608Metric" (at 228.727 151.765 90)
       (effects (font (size 1.27 1.27)) hide)
     )
@@
       (effects (font (size 1.27 1.27)) (justify left))
     )
-    (property "Footprint" "" (at 146.812 66.675 90)
+    (property "Footprint" "Resistor_SMD:R_0603_1608Metric" (at 146.812 66.675 90)
       (effects (font (size 1.27 1.27)) hide)
     )
@@
       (effects (font (size 1.27 1.27)))
     )
-    (property "Footprint" "" (at 78.105 142.24 0)
+    (property "Footprint" "components:HDSP_DIP12" (at 78.105 142.24 0)
       (effects (font (size 1.27 1.27)) hide)
     )
@@
       (effects (font (size 1.27 1.27)))
     )
-    (property "Footprint" "" (at 40.005 49.1998 0)
-      (effects (font (size 1.27 1.27)) hide)
-    )
+    (property "Footprint" "Capacitor_SMD:C_0603_1608Metric" (at 40.005 49.1998 0)
+      (effects (font (size 1.27 1.27)) hide)
+    )

Commit message: minor fixes in vqc10_x10 and hdsp2000_x20 pcb/schematics
Parts:
- Q2, Q3, Q4, Q5, Q6: value DMP2022LSS -> SQ4435EY
Changed lines of the file:
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@@
       (effects (font (size 1.27 1.27)) (justify left))
     )
-    (property "Value" "DMP2022LSS" (at 137.16 152.4 0)
+    (property "Value" "SQ4435EY" (at 137.16 152.4 0)
       (effects (font (size 1.27 1.27)) (justify left))
     )
@@
       (effects (font (size 1.27 1.27)) (justify left))
     )
-    (property "Value" "DMP2022LSS" (at 136.525 100.33 0)
+    (property "Value" "SQ4435EY" (at 136.525 100.33 0)
       (effects (font (size 1.27 1.27)) (justify left))
     )
@@
       (effects (font (size 1.27 1.27)) (justify left))
     )
-    (property "Value" "DMP2022LSS" (at 135.255 47.625 0)
+    (property "Value" "SQ4435EY" (at 135.255 47.625 0)
       (effects (font (size 1.27 1.27)) (justify left))
     )
@@
       (effects (font (size 1.27 1.27)) (justify left))
     )
-    (property "Value" "DMP2022LSS" (at 137.16 126.365 0)
+    (property "Value" "SQ4435EY" (at 137.16 126.365 0)
       (effects (font (size 1.27 1.27)) (justify left))
     )
@@
       (effects (font (size 1.27 1.27)) (justify left))
     )
-    (property "Value" "DMP2022LSS" (at 135.89 74.295 0)
-      (effects (font (size 1.27 1.27)) (justify left))
-    )
+    (property "Value" "SQ4435EY" (at 135.89 74.295 0)
+      (effects (font (size 1.27 1.27)) (justify left))
+    )
