File: hardware/vin_display_hdsp2000_x20/vin_display_hdsp2000_x20.kicad_pcb (KiCad board)
At the start: 4 copper layers, 170 x 50 mm, 104 parts, among them J1 DEBUG, J2 USB_B_Micro, J3 DEBUG_UART, J4 IF_UART, J5 AUX_CONNECTOR, Q1 BSS138, Q2 DMP2022LSS, Q3 DMP2022LSS, Q4 DMP2022LSS, Q5 DMP2022LSS, Q6 DMP2022LSS, SW1 SW_RESET, SW2 BOOTSEL, SW3 KNOB, U1 W25Q16JVSNIQ, U10 HDSP-2000, U11 HDSP-2000, U12 HDSP-2000, U13 HDSP-2000, U14 HDSP-2000, U15 HDSP-2000, U16 HDSP-2000, U17 HDSP-2000, U18 HDSP-2000, U19 HDSP-2000, U2 MIC23050-SYML, U20 HDSP-2000, U21 HDSP-2000, U22 HDSP-2000, U23 HDSP-2000, U24 HDSP-2000, U3 RP2040, U5 HDSP-2000, U6 HDSP-2000, U7 HDSP-2000, U8 HDSP-2000, U9 HDSP-2000, X1 12MHz

Commit message: route hdsp2000_x20 board
Parts:
- added D3: D, components:Diode_TO252, F.Cu at (144.2, 121.7)
- added F1: 10A, components:Fuse_2410, F.Cu at (149.7, 119.8)
- added J6: Conn_01x02, components:Conn_2x3_96, F.Cu at (154.2, 125.2)
- added Q7: DMG2301L, Package_TO_SOT_SMD:SOT-23, F.Cu at (150.4, 80.9)
- added R13: 100K, Resistor_SMD:R_0603_1608Metric, F.Cu at (147.4, 81.1)
- J1, J3: footprint Connector_PinHeader_2.54mm:PinHeader_1x03_P2.54mm_Vertical -> Connector_JST:JST_EH_B3B-EH-A_1x03_P2.50mm_Vertical
- J4: footprint Connector_PinHeader_2.54mm:PinHeader_1x04_P2.54mm_Vertical -> Connector_JST:JST_EH_B4B-EH-A_1x04_P2.50mm_Vertical
- JP1: footprint Jumper:SolderJumper-3_P1.3mm_Open_Pad1.0x1.5mm -> components:Solder_jumber_3pad
- moved C23 233.0 mm to (241.4, 82.8)
- moved C28 232.6 mm to (241.7, 93.0)
- moved C29 223.0 mm to (231.2, 92.2), turned to 180 degrees
- moved C24 222.5 mm to (231.4, 82.1), turned to 180 degrees
- moved C33 211.7 mm to (241.6, 103.1)
- moved C38 210.5 mm to (241.5, 113.4)
- moved C30 205.6 mm to (213.4, 92.3), turned to 180 degrees
- moved C25 204.8 mm to (213.5, 82.2), turned to 180 degrees
- moved C39 204.4 mm to (231.4, 112.5), turned to 180 degrees
- moved C34 201.1 mm to (231.4, 102.3)
- moved C31 188.2 mm to (195.5, 92.2), turned to 180 degrees
- moved C40 188.1 mm to (213.4, 112.5), turned to 180 degrees
- moved C26 187.1 mm to (195.5, 82.1), turned to 180 degrees
- moved C35 184.4 mm to (213.5, 102.3), turned to 180 degrees
- moved C41 172.3 mm to (195.5, 112.5), turned to 180 degrees
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Connections:
- J5 pad 4: GND -> GP14
- J5 pad 6: GND -> GP15
Routing:
- net DISP_VCC: track 0.00 -> 516.8 mm, vias 0 -> 6
- net DRV_COL1: track 113.8 -> 469.9 mm, vias 8 -> 21
- net DISP_CLK: track 33.2 -> 389.1 mm, vias 2 -> 1
- net DRV_COL2: track 108.3 -> 450.5 mm, vias 8 -> 24
- net DRV_COL3: track 101.9 -> 420.1 mm, vias 8 -> 16
- net DRV_COL4: track 95.7 -> 392.7 mm, vias 8 -> 23
- net DRV_COL5: track 88.8 -> 372.0 mm, vias 0 -> 6
- net DISP_VB: track 0.00 -> 256.8 mm, vias 0 -> 1
- net VSYS: track 280.4 -> 113.5 mm, vias 2 -> 5
- net DISP_DATA: track 23.9 -> 133.0 mm, vias 2 -> 1
- net D5_DOUT: track 0.00 -> 97.5 mm
- net D15_DOUT: track 0.00 -> 95.8 mm
- net (no net): track 92.5 -> 0.00 mm
- net Net-(JP1-C): track 0.00 -> 80.7 mm, vias 0 -> 1
- net KNOB_SW: track 70.8 -> 129.1 mm
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- added copper zone on F.Cu, net DISP_VCC
- added copper zone on F.Cu, net VSYS
Other:
- board size 170 x 50 mm -> 148 x 52 mm
- board text added: "CoolHorse Industries 2024"
- board text added: "VinDisplay hdsp2000_x20 v1.0"
- board text removed: "CoolHorse Industries 2023"
- board text removed: "VinDisplay hdsp2112_x6 v1.0"

Commit message: hdsp2000_x20 pcb v1.0
Other:
- board text added: "DIO/GNF/CLK"
- board text added: "RX/GND/TX"
- board text added: "RX/GND/TX/VSYS"
- board text removed: "CLK/GND/DIO"
- board text removed: "TX/GND/RX"
- board text removed: "VSYS/TX/GND/RX"

Commit message: hdsp2000_x20 minor changes
Connections:
- U3 pad 16: GP13 -> unconnected-(U3-GPIO13-Pad16)
- U3 pad 27: GP16 -> unconnected-(U3-GPIO16-Pad27)
- U3 pad 28: GP17 -> unconnected-(U3-GPIO17-Pad28)
- U3 pad 29: GP18 -> unconnected-(U3-GPIO18-Pad29)
- U3 pad 30: GP19 -> unconnected-(U3-GPIO19-Pad30)
- U3 pad 31: GP20 -> unconnected-(U3-GPIO20-Pad31)
- U3 pad 32: GP21 -> unconnected-(U3-GPIO21-Pad32)
- U3 pad 34: GP22 -> unconnected-(U3-GPIO22-Pad34)
- U3 pad 35: GP23 -> unconnected-(U3-GPIO23-Pad35)
Changed lines of the file:
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@@
       (drillshape 0)
       (scaleselection 1)
-      (outputdirectory "vindisp_hdsp2112_x6_gerbers/")
+      (outputdirectory "./gerbers")
     )
   )
@@
   (net 58 "DISP_DATA")
   (net 59 "DISP_BR")
-  (net 60 "GP13")
+  (net 60 "unconnected-(U3-GPIO13-Pad16)")
   (net 61 "GP14")
   (net 62 "GP15")
-  (net 63 "GP16")
-  (net 64 "GP17")
-  (net 65 "GP18")
-  (net 66 "GP19")
-  (net 67 "GP20")
-  (net 68 "GP21")
-  (net 69 "GP22")
-  (net 70 "GP23")
+  (net 63 "unconnected-(U3-GPIO16-Pad27)")
+  (net 64 "unconnected-(U3-GPIO17-Pad28)")
+  (net 65 "unconnected-(U3-GPIO18-Pad29)")
+  (net 66 "unconnected-(U3-GPIO19-Pad30)")
+  (net 67 "unconnected-(U3-GPIO20-Pad31)")
+  (net 68 "unconnected-(U3-GPIO21-Pad32)")
+  (net 69 "unconnected-(U3-GPIO22-Pad34)")
+  (net 70 "unconnected-(U3-GPIO23-Pad35)")
   (net 71 "unconnected-(U5-NC-Pad6)")
   (net 72 "Net-(U5-DOUT)")
@@
     (fp_line (start 10 2.2) (end 10 -1.6)
       (stroke (width 0.1) (type solid)) (layer "F.Fab"))
-    (pad "1" thru_hole roundrect (at 0 0 180) (size 1.7 1.95) (drill 0.95) (layers "*.Cu" "*.Mask") (roundrect_rratio 0.147059)
+    (pad "1" thru_hole roundrect (at 0 0 180) (size 1.7 1.95) (drill 0.95) (layers "*.Cu" "*.Mask") (roundrect_rratio 0.1470588235)
       (net 3 "VSYS") (pinfunction "Pin_1") (pintype "passive"))
     (pad "2" thru_hole oval (at 2.5 0 180) (size 1.7 1.95) (drill 0.95) (layers "*.Cu" "*.Mask")
@@
     (fp_line (start 7.5 2.2) (end 7.5 -1.6)
       (stroke (width 0.1) (type solid)) (layer "F.Fab"))
-    (pad "1" thru_hole roundrect (at 0 0 180) (size 1.7 1.95) (drill 0.95) (layers "*.Cu" "*.Mask") (roundrect_rratio 0.147059)
+    (pad "1" thru_hole roundrect (at 0 0 180) (size 1.7 1.95) (drill 0.95) (layers "*.Cu" "*.Mask") (roundrect_rratio 0.1470588235)
       (net 18 "UART0_TX") (pinfunction "Pin_1") (pintype "passive"))
     (pad "2" thru_hole oval (at 2.5 0 180) (size 1.7 1.95) (drill 0.95) (layers "*.Cu" "*.Mask")
@@
       (net 59 "DISP_BR") (pinfunction "GPIO12") (pintype "bidirectional"))
     (pad "16" smd roundrect (at -2.2 3.4375 180) (size 0.2 0.875) (layers "F.Cu" "F.Paste" "F.Mask") (roundrect_rratio 0.25)
-      (net 60 "GP13") (pinfunction "GPIO13") (pintype "bidirectional"))
+      (net 60 "unconnected-(U3-GPIO13-Pad16)") (pinfunction "GPIO13") (pintype "bidirectional+no_connect"))
     (pad "17" smd roundrect (at -1.8 3.4375 180) (size 0.2 0.875) (layers "F.Cu" "F.Paste" "F.Mask") (roundrect_rratio 0.25)
       (net 61 "GP14") (pinfunction "GPIO14") (pintype "bidirectional"))
@@
       (net 32 "Net-(U3-RUN)") (pinfunction "RUN") (pintype "input"))
     (pad "27" smd roundrect (at 2.2 3.4375 180) (size 0.2 0.875) (layers "F.Cu" "F.Paste" "F.Mask") (roundrect_rratio 0.25)
-      (net 63 "GP16") (pinfunction "GPIO16") (pintype "bidirectional"))
+      (net 63 "unconnected-(U3-GPIO16-Pad27)") (pinfunction "GPIO16") (pintype "bidirectional+no_connect"))
     (pad "28" smd roundrect (at 2.6 3.4375 180) (size 0.2 0.875) (layers "F.Cu" "F.Paste" "F.Mask") (roundrect_rratio 0.25)
-      (net 64 "GP17") (pinfunction "GPIO17") (pintype "bidirectional"))
+      (net 64 "unconnected-(U3-GPIO17-Pad28)") (pinfunction "GPIO17") (pintype "bidirectional+no_connect"))
     (pad "29" smd roundrect (at 3.4375 2.6 180) (size 0.875 0.2) (layers "F.Cu" "F.Paste" "F.Mask") (roundrect_rratio 0.25)
-      (net 65 "GP18") (pinfunction "GPIO18") (pintype "bidirectional"))
+      (net 65 "unconnected-(U3-GPIO18-Pad29)") (pinfunction "GPIO18") (pintype "bidirectional+no_connect"))
     (pad "30" smd roundrect (at 3.4375 2.2 180) (size 0.875 0.2) (layers "F.Cu" "F.Paste" "F.Mask") (roundrect_rratio 0.25)
-      (net 66 "GP19") (pinfunction "GPIO19") (pintype "bidirectional"))
+      (net 66 "unconnected-(U3-GPIO19-Pad30)") (pinfunction "GPIO19") (pintype "bidirectional+no_connect"))
     (pad "31" smd roundrect (at 3.4375 1.8 180) (size 0.875 0.2) (layers "F.Cu" "F.Paste" "F.Mask") (roundrect_rratio 0.25)
-      (net 67 "GP20") (pinfunction "GPIO20") (pintype "bidirectional"))
+      (net 67 "unconnected-(U3-GPIO20-Pad31)") (pinfunction "GPIO20") (pintype "bidirectional+no_connect"))
     (pad "32" smd roundrect (at 3.4375 1.4 180) (size 0.875 0.2) (layers "F.Cu" "F.Paste" "F.Mask") (roundrect_rratio 0.25)
-      (net 68 "GP21") (pinfunction "GPIO21") (pintype "bidirectional"))
+      (net 68 "unconnected-(U3-GPIO21-Pad32)") (pinfunction "GPIO21") (pintype "bidirectional+no_connect"))
     (pad "33" smd roundrect (at 3.4375 1 180) (size 0.875 0.2) (layers "F.Cu" "F.Paste" "F.Mask") (roundrect_rratio 0.25)
       (net 6 "3V3") (pinfunction "IOVDD") (pintype "passive"))
     (pad "34" smd roundrect (at 3.4375 0.6 180) (size 0.875 0.2) (layers "F.Cu" "F.Paste" "F.Mask") (roundrect_rratio 0.25)
-      (net 69 "GP22") (pinfunction "GPIO22") (pintype "bidirectional"))
+      (net 69 "unconnected-(U3-GPIO22-Pad34)") (pinfunction "GPIO22") (pintype "bidirectional+no_connect"))
     (pad "35" smd roundrect (at 3.4375 0.2 180) (size 0.875 0.2) (layers "F.Cu" "F.Paste" "F.Mask") (roundrect_rratio 0.25)
-      (net 70 "GP23") (pinfunction "GPIO23") (pintype "bidirectional"))
+      (net 70 "unconnected-(U3-GPIO23-Pad35)") (pinfunction "GPIO23") (pintype "bidirectional+no_connect"))
     (pad "36" smd roundrect (at 3.4375 -0.2 180) (size 0.875 0.2) (layers "F.Cu" "F.Paste" "F.Mask") (roundrect_rratio 0.25)
       (net 9 "KNOB_SW") (pinfunction "GPIO24") (pintype "bidirectional"))
@@
     (fp_line (start 7.5 2.2) (end 7.5 -1.6)
       (stroke (width 0.1) (type solid)) (layer "F.Fab"))
-    (pad "1" thru_hole roundrect (at 0 0 180) (size 1.7 1.95) (drill 0.95) (layers "*.Cu" "*.Mask") (roundrect_rratio 0.147059)
+    (pad "1" thru_hole roundrect (at 0 0 180) (size 1.7 1.95) (drill 0.95) (layers "*.Cu" "*.Mask") (roundrect_rratio 0.1470588235)
       (net 14 "SWCLK") (pinfunction "Pin_1") (pintype "passive"))
     (pad "2" thru_hole oval (at 2.5 0 180) (size 1.7 1.95) (drill 0.95) (layers "*.Cu" "*.Mask")

Commit message: minor fixes in vqc10_x10 and hdsp2000_x20 pcb/schematics
Parts:
- Q2, Q3, Q4, Q5, Q6: value DMP2022LSS -> SQ4435EY
Changed lines of the file:
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@@
         (effects (font (size 1 1) (thickness 0.1)))
     )
-    (fp_text value "DMP2022LSS" (at 2.54 2.54 -90 unlocked) (layer "F.Fab") hide
+    (fp_text value "SQ4435EY" (at 2.54 2.54 -90 unlocked) (layer "F.Fab") hide
         (effects (font (size 1 1) (thickness 0.15)))
     )
@@
         (effects (font (size 1 1) (thickness 0.1)))
     )
-    (fp_text value "DMP2022LSS" (at 2.54 2.54 -90 unlocked) (layer "F.Fab") hide
+    (fp_text value "SQ4435EY" (at 2.54 2.54 -90 unlocked) (layer "F.Fab") hide
         (effects (font (size 1 1) (thickness 0.15)))
     )
@@
         (effects (font (size 1 1) (thickness 0.1)))
     )
-    (fp_text value "DMP2022LSS" (at 2.54 2.54 -90 unlocked) (layer "F.Fab") hide
+    (fp_text value "SQ4435EY" (at 2.54 2.54 -90 unlocked) (layer "F.Fab") hide
         (effects (font (size 1 1) (thickness 0.15)))
     )
@@
         (effects (font (size 1 1) (thickness 0.1)))
     )
-    (fp_text value "DMP2022LSS" (at 2.54 2.54 -90 unlocked) (layer "F.Fab") hide
+    (fp_text value "SQ4435EY" (at 2.54 2.54 -90 unlocked) (layer "F.Fab") hide
         (effects (font (size 1 1) (thickness 0.15)))
     )
@@
         (effects (font (size 1 1) (thickness 0.1)))
     )
-    (fp_text value "DMP2022LSS" (at 2.54 2.54 -90 unlocked) (layer "F.Fab") hide
+    (fp_text value "SQ4435EY" (at 2.54 2.54 -90 unlocked) (layer "F.Fab") hide
         (effects (font (size 1 1) (thickness 0.15)))
     )
