File: hardware/vin_display_vqc10_x10/displays.kicad_sch (KiCad schematic)
At the start: 10 parts, among them U10 VQC10, U11 VQC10, U12 VQC10, U13 VQC10, U4 VQC10, U5 VQC10, U6 VQC10, U7 VQC10, U8 VQC10, U9 VQC10

Commit message: routing vqc10_x10
Parts:
- U10, U11, U12, U13, U4, U5, U6, U7, U8, U9: footprint (none) -> components:VQC10
Connections:
- net DISP_VCC: now reaches U4.14 (VCC), U5.14 (VCC), U6.14 (VCC), U7.14 (VCC), U8.14 (VCC)
- net DISP_VCC: now also U10.14 (VCC), U11.14 (VCC), U12.14 (VCC), U13.14 (VCC), U9.14 (VCC)
Changed lines of the file:
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@@
   (junction (at 159.385 142.24) (diameter 0) (color 0 0 0 0)
   )
+  (junction (at 71.12 71.755) (diameter 0) (color 0 0 0 0)
+  )
   (junction (at 243.205 149.86) (diameter 0) (color 0 0 0 0)
   )
@@
   )
   (junction (at 149.225 101.6) (diameter 0) (color 0 0 0 0)
+  )
+  (junction (at 70.485 147.32) (diameter 0) (color 0 0 0 0)
   )
   (junction (at 182.245 134.62) (diameter 0) (color 0 0 0 0)
@@
     (stroke (width 0) (type default))
   )
+  (wire (pts (xy 29.21 147.32) (xy 70.485 147.32))
+    (stroke (width 0) (type default))
+  )
   (wire (pts (xy 144.145 104.14) (xy 144.145 112.395))
     (stroke (width 0) (type default))
@@
     (stroke (width 0) (type default))
   )
+  (wire (pts (xy 29.845 71.755) (xy 71.12 71.755))
+    (stroke (width 0) (type default))
+  )
   (wire (pts (xy 48.26 36.195) (xy 48.26 28.575))
     (stroke (width 0) (type default))
@@
     )
   )
+  (global_label "DISP_VCC" (shape input) (at 29.845 71.755 180) (fields_autoplaced)
+    (effects (font (size 1.27 1.27)) (justify right))
+    (property "Intersheetrefs" "${INTERSHEET_REFS}" (at 17.9093 71.755 0)
+      (effects (font (size 1.27 1.27)) (justify right) hide)
+    )
+  )
   (global_label "DRV_R5" (shape input) (at 29.21 106.68 180) (fields_autoplaced)
     (effects (font (size 1.27 1.27)) (justify right))
@@
     (effects (font (size 1.27 1.27)) (justify right))
     (property "Intersheetrefs" "${INTERSHEET_REFS}" (at 19.7841 26.035 0)
+      (effects (font (size 1.27 1.27)) (justify right) hide)
+    )
+  )
+  (global_label "DISP_VCC" (shape input) (at 29.21 147.32 180) (fields_autoplaced)
+    (effects (font (size 1.27 1.27)) (justify right))
+    (property "Intersheetrefs" "${INTERSHEET_REFS}" (at 17.2743 147.32 0)
       (effects (font (size 1.27 1.27)) (justify right) hide)
     )
@@
       (effects (font (size 1.27 1.27)) (justify left))
     )
-    (property "Footprint" "" (at 144.78 46.99 0)
+    (property "Footprint" "components:VQC10" (at 144.78 46.99 0)
       (effects (font (size 1.27 1.27)) hide)
     )
@@
       (effects (font (size 1.27 1.27)) (justify left))
     )
-    (property "Footprint" "" (at 241.3 46.99 0)
+    (property "Footprint" "components:VQC10" (at 241.3 46.99 0)
       (effects (font (size 1.27 1.27)) hide)
     )
@@
       (effects (font (size 1.27 1.27)) (justify left))
     )
-    (property "Footprint" "" (at 48.26 46.355 0)
+    (property "Footprint" "components:VQC10" (at 48.26 46.355 0)
       (effects (font (size 1.27 1.27)) hide)
     )
@@
       (effects (font (size 1.27 1.27)) (justify left))
     )
-    (property "Footprint" "" (at 95.885 121.92 0)
+    (property "Footprint" "components:VQC10" (at 95.885 121.92 0)
       (effects (font (size 1.27 1.27)) hide)
     )
@@
       (effects (font (size 1.27 1.27)) (justify left))
     )
-    (property "Footprint" "" (at 193.04 46.99 0)
+    (property "Footprint" "components:VQC10" (at 193.04 46.99 0)
       (effects (font (size 1.27 1.27)) hide)
     )
@@
       (effects (font (size 1.27 1.27)) (justify left))
     )
-    (property "Footprint" "" (at 96.52 46.355 0)
+    (property "Footprint" "components:VQC10" (at 96.52 46.355 0)
       (effects (font (size 1.27 1.27)) hide)
     )
@@
       (effects (font (size 1.27 1.27)) (justify left))
     )
-    (property "Footprint" "" (at 240.665 122.555 0)
+    (property "Footprint" "components:VQC10" (at 240.665 122.555 0)
       (effects (font (size 1.27 1.27)) hide)
     )
@@
       (effects (font (size 1.27 1.27)) (justify left))
     )
-    (property "Footprint" "" (at 144.145 122.555 0)
+    (property "Footprint" "components:VQC10" (at 144.145 122.555 0)
       (effects (font (size 1.27 1.27)) hide)
     )
@@
       (effects (font (size 1.27 1.27)) (justify left))
     )
-    (property "Footprint" "" (at 192.405 122.555 0)
+    (property "Footprint" "components:VQC10" (at 192.405 122.555 0)
       (effects (font (size 1.27 1.27)) hide)
     )
@@
       (effects (font (size 1.27 1.27)) (justify left))
     )
-    (property "Footprint" "" (at 47.625 121.92 0)
-      (effects (font (size 1.27 1.27)) hide)
-    )
+    (property "Footprint" "components:VQC10" (at 47.625 121.92 0)
+      (effects (font (size 1.27 1.27)) hide)
+    )
