File: hardware/vin_display_vqc10_x10/vin_display_vqc10_x10.kicad_sch (KiCad schematic)
At the start: 56 parts, among them J1 DEBUG, J2 USB_B_Micro, J3 DEBUG_UART, J4 IF_UART, J5 AUX_CONNECTOR, J6 Conn_01x02, Q1 BSS138, Q7 DMG2301L, SW1 SW_RESET, SW2 BOOTSEL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

Commit message: routing vqc10_x10
Parts:
- removed Q7: DMG2301L, Package_TO_SOT_SMD:SOT-23, symbol Transistor_FET:DMG2301L
- removed R13: 100K, Resistor_SMD:R_0603_1608Metric, symbol Device:R
Changed lines of the file:
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@@
   (junction (at 214.63 118.11) (diameter 0) (color 0 0 0 0)
-  )
-  (junction (at 259.715 89.535) (diameter 0) (color 0 0 0 0)
   )
   (junction (at 119.38 152.4) (diameter 0) (color 0 0 0 0)
@@
     (stroke (width 0) (type default))
   )
-  (wire (pts (xy 269.875 76.835) (xy 271.78 76.835))
-    (stroke (width 0) (type default))
-  )
-  (wire (pts (xy 254.635 89.535) (xy 259.715 89.535))
-    (stroke (width 0) (type default))
-  )
   (wire (pts (xy 267.97 107.95) (xy 252.73 107.95))
     (stroke (width 0) (type default))
@@
     (stroke (width 0) (type default))
   )
-  (wire (pts (xy 269.875 94.615) (xy 269.875 97.155))
-    (stroke (width 0) (type default))
-  )
   (wire (pts (xy 134.62 166.37) (xy 149.86 166.37))
     (stroke (width 0) (type default))
@@
     (stroke (width 0) (type default))
   )
-  (wire (pts (xy 269.875 84.455) (xy 269.875 76.835))
-    (stroke (width 0) (type default))
-  )
   (wire (pts (xy 204.47 45.72) (xy 204.47 50.8))
     (stroke (width 0) (type default))
@@
     (stroke (width 0) (type default))
   )
-  (wire (pts (xy 254.635 76.2) (xy 259.715 76.2))
-    (stroke (width 0) (type default))
-  )
   (wire (pts (xy 102.87 96.52) (xy 102.87 92.71))
     (stroke (width 0) (type default))
@@
     (stroke (width 0) (type default))
   )
-  (wire (pts (xy 262.255 89.535) (xy 259.715 89.535))
-    (stroke (width 0) (type default))
-  )
   (wire (pts (xy 100.33 147.32) (xy 102.87 147.32))
     (stroke (width 0) (type default))
@@
     (stroke (width 0) (type default))
   )
-  (wire (pts (xy 259.715 78.74) (xy 259.715 76.2))
-    (stroke (width 0) (type default))
-  )
   (wire (pts (xy 196.85 156.21) (xy 186.69 156.21))
     (stroke (width 0) (type default))
@@
     (stroke (width 0) (type default))
   )
-  (wire (pts (xy 269.875 97.155) (xy 271.78 97.155))
-    (stroke (width 0) (type default))
-  )
   (wire (pts (xy 237.49 22.86) (xy 237.49 25.4))
     (stroke (width 0) (type default))
@@
   )
   (wire (pts (xy 260.35 62.865) (xy 250.19 62.865))
-    (stroke (width 0) (type default))
-  )
-  (wire (pts (xy 259.715 89.535) (xy 259.715 86.36))
     (stroke (width 0) (type default))
   )
@@
     )
   )
-  (global_label "3V3" (shape input) (at 254.635 76.2 180) (fields_autoplaced)
-    (effects (font (size 1.27 1.27)) (justify right))
-    (property "Intersheetrefs" "${INTERSHEET_REFS}" (at 248.1422 76.2 0)
-      (effects (font (size 1.27 1.27)) (justify right) hide)
-    )
-  )
   (global_label "UART1_RX" (shape input) (at 181.61 62.23 0) (fields_autoplaced)
     (effects (font (size 1.27 1.27)) (justify left))
     (property "Intersheetrefs" "${INTERSHEET_REFS}" (at 193.3364 62.1506 0)
       (effects (font (size 1.27 1.27)) (justify left) hide)
-    )
-  )
-  (global_label "DISP_BR" (shape input) (at 254.635 89.535 180) (fields_autoplaced)
-    (effects (font (size 1.27 1.27)) (justify right))
-    (property "Intersheetrefs" "${INTERSHEET_REFS}" (at 243.7879 89.535 0)
-      (effects (font (size 1.27 1.27)) (justify right) hide)
     )
   )
@@
     (property "Intersheetrefs" "${INTERSHEET_REFS}" (at 238.8893 48.26 0)
       (effects (font (size 1.27 1.27)) (justify right) hide)
-    )
-  )
-  (global_label "DISP_VCC" (shape input) (at 271.78 97.155 0) (fields_autoplaced)
-    (effects (font (size 1.27 1.27)) (justify left))
-    (property "Intersheetrefs" "${INTERSHEET_REFS}" (at 283.7157 97.155 0)
-      (effects (font (size 1.27 1.27)) (justify left) hide)
-    )
-  )
-  (global_label "DISP_VB" (shape input) (at 271.78 76.835 0) (fields_autoplaced)
-    (effects (font (size 1.27 1.27)) (justify left))
-    (property "Intersheetrefs" "${INTERSHEET_REFS}" (at 282.4457 76.835 0)
-      (effects (font (size 1.27 1.27)) (justify left) hide)
     )
   )
@@
         (path "/d55a26ad-800d-41cd-b8dc-29004e00bfdd"
           (reference "#PWR0109") (unit 1)
-        )
-      )
-    )
-  )
-  (symbol (lib_id "Transistor_FET:DMG2301L") (at 267.335 89.535 0) (unit 1)
-    (in_bom yes) (on_board yes) (dnp no) (fields_autoplaced)
-    (property "Reference" "Q7" (at 273.05 88.265 0)
-      (effects (font (size 1.27 1.27)) (justify left))
-    )
-    (property "Value" "DMG2301L" (at 273.05 90.805 0)
-      (effects (font (size 1.27 1.27)) (justify left))
-    )
-    (property "Footprint" "Package_TO_SOT_SMD:SOT-23" (at 272.415 91.44 0)
-      (effects (font (size 1.27 1.27) italic) (justify left) hide)
-    )
-    (property "Datasheet" "https://www.diodes.com/assets/Datasheets/DMG2301L.pdf" (at 267.335 89.535 0)
-      (effects (font (size 1.27 1.27)) (justify left) hide)
-    )
-    (pin "3")
-    (pin "1")
-    (pin "2")
-    (instances
-      (project "vin_display_vqc10_x10"
-        (path "/d55a26ad-800d-41cd-b8dc-29004e00bfdd"
-          (reference "Q7") (unit 1)
         )
       )
@@
         )
       )
-    )
-  )
-  (symbol (lib_id "Device:R") (at 259.715 82.55 0) (unit 1)
-    (in_bom yes) (on_board yes) (dnp no) (fields_autoplaced)
-    (property "Reference" "R13" (at 261.62 81.28 0)
-      (effects (font (size 1.27 1.27)) (justify left))
-    )
-    (property "Value" "100K" (at 261.62 83.82 0)
-      (effects (font (size 1.27 1.27)) (justify left))
-    )
-    (property "Footprint" "Resistor_SMD:R_0603_1608Metric" (at 257.937 82.55 90)
-      (effects (font (size 1.27 1.27)) hide)
-    )
-    (property "Datasheet" "~" (at 259.715 82.55 0)
-      (effects (font (size 1.27 1.27)) hide)
-    )
-    (pin "1")
-    (pin "2")
-    (instances
-      (project "vin_display_vqc10_x10"
-        (path "/d55a26ad-800d-41cd-b8dc-29004e00bfdd"
-          (reference "R13") (unit 1)
-        )
-      )
