File: hardware/vin_display_vqc10_x10/vin_display_vqc10_x10.kicad_pcb (KiCad board)
At the start: 4 copper layers, 242 x 55 mm, 92 parts, among them J1 DEBUG, J2 USB_B_Micro, J3 DEBUG_UART, J4 IF_UART, J5 AUX_CONNECTOR, J6 Conn_01x02, Q1 BSS138, Q2 DMP2022LSS, Q3 DMP2022LSS, Q4 DMP2022LSS, Q5 DMP2022LSS, Q6 DMP2022LSS, Q8 DMP2022LSS, Q9 DMP2022LSS, SW1 SW_RESET, SW2 BOOTSEL, SW3 KNOB, U1 W25Q16JVSNIQ, U10 VQC10, U11 VQC10, U12 VQC10, U13 VQC10, U14 74HCT154, U15 74HCT154, U16 74HCT154, U2 MIC23050-SYML, U3 RP2040, U4 VQC10, U5 VQC10, U6 VQC10, U7 VQC10, U8 VQC10, U9 VQC10, X1 12MHz

Commit message: minor fixes in vqc10_x10 and hdsp2000_x20 pcb/schematics
Other:
- board text added: "VinDisplay vqc10_x10 v1.0"
- board text removed: "VinDisplay hdsp2000_x20 v1.0"
Changed lines of the file:
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@@
     (property "ki_keywords" "R res resistor")
     (attr smd)
-    (fp_text reference "R17" (at -3.3528 13.1064 90) (layer "F.SilkS")
+    (fp_text reference "R17" (at -3.3528 13.1064 90) (layer "F.SilkS") hide
         (effects (font (size 0.7 0.7) (thickness 0.15)))
     )
@@
     (property "ki_keywords" "R res resistor")
     (attr smd)
-    (fp_text reference "R19" (at -3.4544 7.5692 90) (layer "F.SilkS")
+    (fp_text reference "R19" (at -3.4544 7.5692 90) (layer "F.SilkS") hide
         (effects (font (size 0.7 0.7) (thickness 0.15)))
     )
@@
     (property "ki_keywords" "R res resistor")
     (attr smd)
-    (fp_text reference "R18" (at -3.3528 8.128 90) (layer "F.SilkS")
+    (fp_text reference "R18" (at -3.3528 8.128 90) (layer "F.SilkS") hide
         (effects (font (size 0.7 0.7) (thickness 0.15)))
     )
@@
     (property "ki_keywords" "R res resistor")
     (attr smd)
-    (fp_text reference "R16" (at -3.302 7.4676 90) (layer "F.SilkS")
+    (fp_text reference "R16" (at -3.302 7.4676 90) (layer "F.SilkS") hide
         (effects (font (size 0.7 0.7) (thickness 0.15)))
     )
@@
     (property "ki_keywords" "R res resistor")
     (attr smd)
-    (fp_text reference "R20" (at -3.4036 14.4272 90) (layer "F.SilkS")
+    (fp_text reference "R20" (at -3.4036 14.4272 90) (layer "F.SilkS") hide
         (effects (font (size 0.7 0.7) (thickness 0.15)))
     )
@@
     (property "ki_keywords" "R res resistor")
     (attr smd)
-    (fp_text reference "R15" (at -3.2512 8.0264 90) (layer "F.SilkS")
+    (fp_text reference "R15" (at -3.2512 8.0264 90) (layer "F.SilkS") hide
         (effects (font (size 0.7 0.7) (thickness 0.15)))
     )
@@
     (property "ki_keywords" "R res resistor")
     (attr smd)
-    (fp_text reference "R21" (at -3.2512 15.494 90) (layer "F.SilkS")
+    (fp_text reference "R21" (at -3.2512 15.494 90) (layer "F.SilkS") hide
         (effects (font (size 0.7 0.7) (thickness 0.15)))
     )
@@
     (effects (font (size 1.5 1.5) (thickness 0.3) bold) (justify left bottom mirror))
   )
-  (gr_text "VinDisplay hdsp2000_x20 v1.0" (at 270.2288 69.3424) (layer "B.SilkS")
+  (gr_text "VinDisplay vqc10_x10 v1.0" (at 270.2288 69.3424) (layer "B.SilkS")
     (effects (font (size 1.5 1.5) (thickness 0.3) bold) (justify left bottom mirror))
   )
